File: Single_transistor_AMP/Single_transistor_AMP.sch (KiCad schematic (older format))
At the start: 10 parts, among them J1 Conn_01x02, J2 Conn_01x02, Q1 BC548

Commit message: Add files via upload
Parts:
- J1, J2: footprint (none) -> TerminalBlock:TerminalBlock_bornier-2_P5.08mm
Changed lines of the file:
@@
 F 0 "J2" H 3668 3075 50  0000 C CNN
 F 1 "Conn_01x02" H 3668 3166 50  0000 C CNN
-F 2 "" H 3750 3400 50  0001 C CNN
+F 2 "TerminalBlock:TerminalBlock_bornier-2_P5.08mm" H 3750 3400 50  0001 C CNN
 F 3 "~" H 3750 3400 50  0001 C CNN
 	1    3750 3400
@@
 F 0 "J1" H 7730 2992 50  0000 L CNN
 F 1 "Conn_01x02" H 7730 2901 50  0000 L CNN
-F 2 "" H 7650 3000 50  0001 C CNN
+F 2 "TerminalBlock:TerminalBlock_bornier-2_P5.08mm" H 7650 3000 50  0001 C CNN
 F 3 "~" H 7650 3000 50  0001 C CNN
 	1    7650 3000
