File: Single_transistor_AMP/Two_transistor_AMP/Two_transistor_AMP.sch (KiCad schematic (older format))
At the start: 14 parts, among them J1 Conn_01x02, J2 Conn_01x02, Q1 Q_NPN_BCE, Q2 Q_NPN_BCE

Commit message: Add files via upload
Parts:
- added J3: 9V, TerminalBlock:TerminalBlock_bornier-2_P5.08mm, symbol Connector_Generic:Conn_01x02
- C2, C3: footprint https:__www.farnell.com_datasheets_2968681.pdf -> Capacitor_THT:CP_Axial_L11.0mm_D6.0mm_P18.00mm_Horizontal
- J1, J2: footprint (none) -> TerminalBlock:TerminalBlock_bornier-2_P5.08mm
Connections:
- net GND: now also J3.1 (Pin_1)
- net +9V: no longer names the net of C3.1, Q2.2 (C), R1.1, R3.1
- net +9V: now also J3.2 (Pin_2)
Changed lines of the file:
@@
 F 0 "C2" V 7998 2500 50  0000 C CNN
 F 1 "0.47uF" V 8089 2500 50  0000 C CNN
-F 2 "https:__www.farnell.com_datasheets_2968681.pdf" H 8288 2350 50  0001 C CNN
+F 2 "Capacitor_THT:CP_Axial_L11.0mm_D6.0mm_P18.00mm_Horizontal" H 8288 2350 50  0001 C CNN
 F 3 "Capacitor_THT:CP_Axial_L11.0mm_D6.0mm_P18.00mm_Horizontal" H 8250 2500 50  0001 C CNN
 	1    8250 2500
@@
 F 0 "C3" H 9615 2396 50  0000 L CNN
 F 1 "47uF" H 9615 2305 50  0000 L CNN
-F 2 "https:__www.farnell.com_datasheets_2968681.pdf" H 9538 2200 50  0001 C CNN
+F 2 "Capacitor_THT:CP_Axial_L11.0mm_D6.0mm_P18.00mm_Horizontal" H 9538 2200 50  0001 C CNN
 F 3 "https://www.farnell.com/datasheets/2968681.pdf" H 9500 2350 50  0001 C CNN
 	1    9500 2350
@@
 Wire Wire Line
 	7550 2150 7550 2000
-Wire Wire Line
-	7550 2000 8350 2000
 Connection ~ 9000 2000
 Wire Wire Line
@@
 F 0 "J2" H 10080 3192 50  0000 L CNN
 F 1 "Conn_01x02" H 10080 3101 50  0000 L CNN
-F 2 "" H 10000 3200 50  0001 C CNN
+F 2 "TerminalBlock:TerminalBlock_bornier-2_P5.08mm" H 10000 3200 50  0001 C CNN
 F 3 "https://www.farnell.com/datasheets/3436052.pdf" H 10000 3200 50  0001 C CNN
 	1    10000 3200
@@
 F 0 "J1" H 6050 2650 50  0000 C CNN
 F 1 "Conn_01x02" V 6200 2850 50  0000 C CNN
-F 2 "" H 6050 2900 50  0001 C CNN
+F 2 "TerminalBlock:TerminalBlock_bornier-2_P5.08mm" H 6050 2900 50  0001 C CNN
 F 3 "~" H 6050 2900 50  0001 C CNN
 	1    6050 2900
@@
 	6300 2800 6250 2800
 $Comp
-L power:+9V #PWR0101
-U 1 1 6182275C
-P 8350 2000
-F 0 "#PWR0101" H 8350 1850 50  0001 C CNN
-F 1 "+9V" H 8365 2173 50  0000 C CNN
-F 2 "" H 8350 2000 50  0001 C CNN
-F 3 "" H 8350 2000 50  0001 C CNN
-	1    8350 2000
-	1    0    0    -1
-$EndComp
+L Connector_Generic:Conn_01x02 J3
+U 1 1 61A105AD
+P 8250 1500
+F 0 "J3" H 8330 1492 50  0000 L CNN
+F 1 "9V" H 8330 1401 50  0000 L CNN
+F 2 "TerminalBlock:TerminalBlock_bornier-2_P5.08mm" H 8250 1500 50  0001 C CNN
+F 3 "https://www.farnell.com/datasheets/3436052.pdf" H 8250 1500 50  0001 C CNN
+	1    8250 1500
+	0    -1   -1   0
+$EndComp
+Wire Wire Line
+	7550 2000 8350 2000
+Wire Wire Line
+	8350 1700 8350 2000
 Connection ~ 8350 2000
 Wire Wire Line
 	8350 2000 9000 2000
+Wire Wire Line
+	8250 1700 8250 1800
+Wire Wire Line
+	8250 1800 8050 1800
+$Comp
+L power:GND #PWR0101
+U 1 1 61A12D74
+P 8050 1800
+F 0 "#PWR0101" H 8050 1550 50  0001 C CNN
+F 1 "GND" V 8055 1672 50  0000 R CNN
+F 2 "" H 8050 1800 50  0001 C CNN
+F 3 "" H 8050 1800 50  0001 C CNN
+	1    8050 1800
+	0    1    1    0
+$EndComp
 $EndSCHEMATC
